File: merope3.kicad_sch (KiCad schematic)
At the start: 71 parts, among them J1 Conn_01x02_Socket, SW1 SW_Push, SW10 SW_Push, SW11 SW_Push, SW12 SW_Push, SW13 SW_Push, SW14 SW_Push, SW15 SW_Push, SW16 SW_Push, SW17 SW_Push, SW18 SW_Push, SW19 SW_Push, SW2 SW_Push, SW20 SW_Push, SW21 SW_Push, SW22 SW_Push, SW23 SW_Push, SW24 SW_Push, SW25 SW_Push, SW26 SW_Push, SW27 SW_Push, SW28 SW_Push, SW29 SW_Push, SW3 SW_Push, SW31 SW_Push, SW32 SW_Push, SW33 SW_Push, SW34 SW_Push, SW35 SW_Push, SW4 SW_Push, SW5 SW_Push, SW6 SW_Push, SW7 SW_Push, SW8 SW_Push, SW9 SW_Push, U1 SuperMini nRF52840

Commit message: almost final
Parts:
- added D37: LED_RGB, LED_SMD:LED_RGB_5050-6, symbol Device:LED_RGB
- added JP1: 3V3 SIDE A, Jumper:SolderJumper-2_P1.3mm_Open_Pad1.0x1.5mm, symbol Jumper:SolderJumper_2_Open
- added JP2: PWR SIDE A, Jumper:SolderJumper-2_P1.3mm_Open_Pad1.0x1.5mm, symbol Jumper:SolderJumper_2_Open
- added JP3: GND SIDE A, Jumper:SolderJumper-2_P1.3mm_Open_Pad1.0x1.5mm, symbol Jumper:SolderJumper_2_Open
- added JP4: 3V3 SIDE B, Jumper:SolderJumper-2_P1.3mm_Open_Pad1.0x1.5mm, symbol Jumper:SolderJumper_2_Open
- added JP5: PWR SIDE B, Jumper:SolderJumper-2_P1.3mm_Open_Pad1.0x1.5mm, symbol Jumper:SolderJumper_2_Open
- added JP6: GND SIDE B, Jumper:SolderJumper-2_P1.3mm_Open_Pad1.0x1.5mm, symbol Jumper:SolderJumper_2_Open
- SW1, SW10, SW11, SW12, SW13, SW14, SW15, SW16, SW17, SW18, SW19, SW2, SW20, SW21, SW22, SW23, SW24, SW25, SW26, SW27, SW28, SW29, SW3, SW4, SW5, SW6, SW7, SW8, SW9: footprint ScottoKeebs_MX:MX_PCB_1.00u -> ScottoKeebs_Scotto:MX_Solder_1.00u_Reversible
- SW30: renamed from SW31; footprint ScottoKeebs_MX:MX_PCB_1.00u -> ScottoKeebs_Scotto:MX_Solder_1.00u_Reversible
- SW31: renamed from SW32; footprint ScottoKeebs_MX:MX_PCB_1.00u -> ScottoKeebs_Scotto:MX_Solder_1.00u_Reversible
- SW32: renamed from SW33; footprint ScottoKeebs_MX:MX_PCB_1.00u -> ScottoKeebs_Scotto:MX_Solder_1.00u_Reversible
- SW33: renamed from SW34; footprint ScottoKeebs_MX:MX_PCB_1.00u -> ScottoKeebs_Scotto:MX_Solder_1.00u_Reversible
- SW34: renamed from SW35; footprint ScottoKeebs_MX:MX_PCB_1.00u -> ScottoKeebs_Scotto:MX_Solder_1.00u_Reversible
Connections:
- net 3V3: now also D37.4 (BA), D37.5 (GA), D37.6 (RA), JP1.2 (B), JP4.2 (B); no longer U1.16 (3V3)
- net GND: now also JP3.2 (B), JP6.2 (B); no longer U1.28 (GND), U1.3 (GND), U1.4 (GND)
- net LED1: now also D37.1 (RK)
- net LED2: now also D37.2 (GK)
- net LED3: now also D37.3 (BK)
- net PWR: now also JP2.2 (B), JP5.2 (B); no longer U1.13 (BAT+), U1.29 (BAT+)
- net BAT REV: now reaches U1.1 (P0.06)
- net BAT REV: now also U1.28 (GND), JP3.1 (A), JP5.1 (A)
- new net 3V3 MAIN: JP1.1 (A), U1.16 (3V3)
- new net 3v3 REV: JP4.1 (A), U1.4 (GND)
- new net BAT MAIN: JP2.1 (A), JP6.1 (A), U1.13 (BAT+), U1.29 (BAT+)

Commit message: updates
Parts:
- added R1, R2, R3: R_Small_US, Resistor_SMD:R_1206_3216Metric_Pad1.30x1.75mm_HandSolder, symbol Device:R_Small_US
Connections:
- net LED1: now also R3.2; no longer D36.1 (RK), D37.1 (RK)
- net LED2: now also R2.2; no longer D36.2 (GK), D37.2 (GK)
- net LED3: now also R1.2; no longer D36.3 (BK), D37.3 (BK)
- new net LED_R1: D36.1 (RK), D37.3 (BK), R3.1
- new net LED_R2: D36.2 (GK), D37.2 (GK), R2.1
- new net LED_R3: D36.3 (BK), D37.1 (RK), R1.1
Other:
- moved on the sheet: D36
