File: merope3.kicad_pcb (KiCad board)
At the start: 2 copper layers, 159.5 x 110.3 mm, 71 parts, among them J1 Conn_01x02_Socket, SW1 SW_Push, SW10 SW_Push, SW11 SW_Push, SW12 SW_Push, SW13 SW_Push, SW14 SW_Push, SW15 SW_Push, SW16 SW_Push, SW17 SW_Push, SW18 SW_Push, SW19 SW_Push, SW2 SW_Push, SW20 SW_Push, SW21 SW_Push, SW22 SW_Push, SW23 SW_Push, SW24 SW_Push, SW25 SW_Push, SW26 SW_Push, SW27 SW_Push, SW28 SW_Push, SW29 SW_Push, SW3 SW_Push, SW31 SW_Push, SW32 SW_Push, SW33 SW_Push, SW34 SW_Push, SW35 SW_Push, SW4 SW_Push, SW5 SW_Push, SW6 SW_Push, SW7 SW_Push, SW8 SW_Push, SW9 SW_Push, U1 SuperMini nRF52840

Commit message: almost final
Parts:
- added D37: LED_RGB, LED_SMD:LED_RGB_5050-6, B.Cu at (170.3, 44.8)
- added JP1: 3V3 SIDE A, Jumper:SolderJumper-2_P1.3mm_Open_Pad1.0x1.5mm, F.Cu at (166.6, 34.0)
- added JP2: PWR SIDE A, Jumper:SolderJumper-2_P1.3mm_Open_Pad1.0x1.5mm, F.Cu at (170.1, 34.0)
- added JP3: GND SIDE A, Jumper:SolderJumper-2_P1.3mm_Open_Pad1.0x1.5mm, F.Cu at (173.7, 34.0)
- added JP4: 3V3 SIDE B, Jumper:SolderJumper-2_P1.3mm_Open_Pad1.0x1.5mm, B.Cu at (173.7, 34.0)
- added JP5: PWR SIDE B, Jumper:SolderJumper-2_P1.3mm_Open_Pad1.0x1.5mm, B.Cu at (170.1, 34.0)
- added JP6: GND SIDE B, Jumper:SolderJumper-2_P1.3mm_Open_Pad1.0x1.5mm, B.Cu at (166.6, 34.0)
- SW1, SW10, SW11, SW12, SW13, SW14, SW15, SW16, SW17, SW18, SW19, SW2, SW20, SW21, SW22, SW23, SW24, SW25, SW26, SW27, SW28, SW29, SW3, SW4, SW5, SW6, SW7, SW8, SW9: footprint ScottoKeebs_MX:MX_PCB_1.00u -> ScottoKeebs_Scotto:MX_Solder_1.00u_Reversible
- SW30: renamed from SW31; footprint ScottoKeebs_MX:MX_PCB_1.00u -> ScottoKeebs_Scotto:MX_Solder_1.00u_Reversible
- SW31: renamed from SW32; footprint ScottoKeebs_MX:MX_PCB_1.00u -> ScottoKeebs_Scotto:MX_Solder_1.00u_Reversible
- SW32: renamed from SW33; footprint ScottoKeebs_MX:MX_PCB_1.00u -> ScottoKeebs_Scotto:MX_Solder_1.00u_Reversible
- SW33: renamed from SW34; footprint ScottoKeebs_MX:MX_PCB_1.00u -> ScottoKeebs_Scotto:MX_Solder_1.00u_Reversible
- SW34: renamed from SW35; footprint ScottoKeebs_MX:MX_PCB_1.00u -> ScottoKeebs_Scotto:MX_Solder_1.00u_Reversible
- moved D36 6.70 mm to (170.3, 44.8)
Connections:
- U1 pad 1: unconnected-(U1-P0.06-Pad1) -> /BAT REV
- U1 pad 13: /PWR -> /BAT MAIN
- U1 pad 16: /3V3 -> /3V3 MAIN
- U1 pad 28: /GND -> /BAT REV
- U1 pad 29: /PWR -> /BAT MAIN
- U1 pad 3: /GND -> unconnected-(U1-GND-Pad3)
- U1 pad 4: /GND -> /3v3 REV
Routing:
- net ROW3: track 216.7 -> 183.3 mm
- net /BAT REV: track 0.00 -> 30.7 mm
- net /BAT MAIN: track 0.00 -> 28.3 mm
- net /GND: track 48.4 -> 26.7 mm, vias 0 -> 2
- net COL4: track 145.5 -> 166.9 mm
- net COL5: track 132.7 -> 154.1 mm
- net /3V3: track 11.2 -> 31.7 mm, vias 0 -> 1
- net ROW0: track 181.1 -> 161.0 mm
- net COL3: track 166.6 -> 185.6 mm
- net COL2: track 167.2 -> 184.8 mm
- net COL1: track 184.8 -> 199.5 mm
- net /LED1: track 5.63 -> 17.8 mm, vias 0 -> 1
- net COL0: track 202.5 -> 214.0 mm
- net /LED3: track 5.61 -> 17.0 mm, vias 0 -> 2
- net COL6: track 103.9 -> 114.0 mm
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Other:
- outline, holes or cut-outs redrawn

Commit message: updates
Parts:
- added R1: R_Small_US, Resistor_SMD:R_1206_3216Metric_Pad1.30x1.75mm_HandSolder, F.Cu at (169.7, 33.0)
- added R2: R_Small_US, Resistor_SMD:R_1206_3216Metric_Pad1.30x1.75mm_HandSolder, F.Cu at (169.7, 36.3)
- added R3: R_Small_US, Resistor_SMD:R_1206_3216Metric_Pad1.30x1.75mm_HandSolder, F.Cu at (169.7, 39.6)
- added REF**: Standoff_M2x4mm, ScottoKeebs_Scotto:Standoff_M2x4mm, F.Cu at (42.9, 89.5)
- added REF**: Standoff_M2x4mm, ScottoKeebs_Scotto:Standoff_M2x4mm, F.Cu at (42.9, 51.4)
- added REF**: Standoff_M2x4mm, ScottoKeebs_Scotto:Standoff_M2x4mm, F.Cu at (138.1, 87.1)
- added REF**: Standoff_M2x4mm, ScottoKeebs_Scotto:Standoff_M2x4mm, F.Cu at (138.1, 49.0)
- moved JP1 6.44 mm to (166.6, 27.5)
- moved JP2 6.44 mm to (170.1, 27.5)
- moved JP3 6.44 mm to (173.7, 27.5)
- moved JP4 6.44 mm to (173.7, 27.5)
- moved JP5 6.44 mm to (170.1, 27.5)
- moved JP6 6.44 mm to (166.6, 27.5)
- moved D37 2.22 mm to (172.5, 45.1), turned to 0 degrees
- moved D36 2.20 mm to (172.4, 45.1), turned to 0 degrees
Connections:
- D36 pad 1: /LED1 -> /LED_R1
- D36 pad 2: /LED2 -> /LED_R2
- D36 pad 3: /LED3 -> /LED_R3
- D37 pad 1: /LED1 -> /LED_R3
- D37 pad 2: /LED2 -> /LED_R2
- D37 pad 3: /LED3 -> /LED_R1
Routing:
- net /LED_R3: track 0.00 -> 22.6 mm, vias 0 -> 1
- net /3V3: track 31.7 -> 53.5 mm, vias 1 -> 2
- net /LED_R2: track 0.00 -> 16.9 mm, vias 0 -> 1
- net /BAT REV: track 30.7 -> 17.7 mm
- net /BAT MAIN: track 28.3 -> 17.1 mm
- net /LED1: track 17.8 -> 6.88 mm, vias 1 -> 0
- net /LED3: track 17.0 -> 7.52 mm, vias 2 -> 0
- net /LED_R1: track 0.00 -> 7.61 mm, vias 0 -> 1
- net /LED2: track 12.1 -> 7.20 mm, vias 2 -> 0
- net /GND: track 26.7 -> 22.3 mm
- net /3v3 REV: track 4.12 -> 8.41 mm
- net /3V3 MAIN: track 4.22 -> 8.45 mm
- net /PWR: track 45.7 -> 47.6 mm
Other:
- board text added: "MEROPE by shoenot github.com/shoenot"

Commit message: final v1.0
Changed lines of the file:
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@@
 		(tags "solder jumper open")
 		(property "Reference" "JP2"
-			(at 0 -1.8 90)
+			(at 2.4125 0 180)
 			(layer "F.SilkS")
 			(effects
@@
 			(at 0 1.9 90)
 			(layer "F.Fab")
+			(hide yes)
 			(effects
 				(font
@@
 		(tags "resistor handsolder")
 		(property "Reference" "R1"
-			(at 0 -1.83 0)
+			(at 0 0 0)
 			(layer "F.SilkS")
 			(effects
@@
 			(at 0 1.83 0)
 			(layer "F.Fab")
+			(hide yes)
 			(effects
 				(font
@@
 		(tags "resistor handsolder")
 		(property "Reference" "R3"
-			(at 0 -1.83 0)
+			(at 0 0 0)
 			(layer "F.SilkS")
 			(effects
@@
 			(at 0 1.83 0)
 			(layer "F.Fab")
+			(hide yes)
 			(effects
 				(font
@@
 		(tags "solder jumper open")
 		(property "Reference" "JP1"
-			(at 0 -1.8 90)
+			(at 2.4125 0 180)
 			(layer "F.SilkS")
 			(effects
@@
 			(at 0 1.9 90)
 			(layer "F.Fab")
+			(hide yes)
 			(effects
 				(font
@@
 		(tags "solder jumper open")
 		(property "Reference" "JP3"
-			(at 0 -1.8 90)
+			(at 2.4125 0 180)
 			(layer "F.SilkS")
 			(effects
@@
 			(at 0 1.9 90)
 			(layer "F.Fab")
+			(hide yes)
 			(effects
 				(font
@@
 		(tags "resistor handsolder")
 		(property "Reference" "R2"
-			(at 0 -1.83 0)
+			(at 0 0 0)
 			(layer "F.SilkS")
 			(effects
@@
 			(at 0 1.83 0)
 			(layer "F.Fab")
+			(hide yes)
 			(effects
 				(font
@@
 		(tags "RGB LED 5050-6")
 		(property "Reference" "D36"
-			(at 0 -3.5 0)
+			(at 0 -0.0575 0)
 			(layer "F.SilkS")
 			(effects
@@
 			(at 0 3.3 0)
 			(layer "F.Fab")
+			(hide yes)
 			(effects
 				(font
@@
 		(tags "solder jumper open")
 		(property "Reference" "JP5"
-			(at 0 1.8 90)
+			(at 2.4125 0 180)
 			(layer "B.SilkS")
 			(effects
@@
 			(at 0 -1.9 90)
 			(layer "B.Fab")
+			(hide yes)
 			(effects
 				(font
@@
 		(tags "solder jumper open")
 		(property "Reference" "JP4"
-			(at 0 1.8 90)
+			(at 2.4125 0 180)
 			(layer "B.SilkS")
 			(effects
@@
 			(at 0 -1.9 90)
 			(layer "B.Fab")
+			(hide yes)
 			(effects
 				(font
@@
 		(tags "RGB LED 5050-6")
 		(property "Reference" "D37"
-			(at 0 3.5 0)
+			(at -0.01875 0 0)
 			(layer "B.SilkS")
 			(effects
@@
 			(at 0 -3.3 0)
 			(layer "B.Fab")
+			(hide yes)
 			(effects
 				(font
@@
 		(tags "solder jumper open")
 		(property "Reference" "JP6"
-			(at 0 1.8 90)
+			(at 2.4125 0 180)
 			(layer "B.SilkS")
 			(effects
@@
 			(at 0 -1.9 90)
 			(layer "B.Fab")
+			(hide yes)
 			(effects
 				(font
@@
 			(layer "B.SilkS")
 			(effects
-				(font
-					(size 1 1)
-					(thickness 0.15)
-				)
-				(justify bottom mirror)
-			)
-		)
-		(fp_text user "1"
-			(at -5.715 13.2825 0)
-			(layer "B.SilkS")
-			(effects
